File: Taller_eagle/taller_2.sch (EAGLE design)
At the start: 10 parts, among them X1 22-23-2021, X2 22-23-2021, X3 22-23-2021

Commit message: carpetas ordenadas y limpias, proyectos de pcbs en este repo
Parts:
- removed LEFTQTR1A, RIGHTQTR1A: (no value), adafruit:PINHD-1X3
- removed QTR8A: (no value), adafruit:PINHD-1X8BIG
- removed S1: (no value), SparkFun-Retired:TAC_SWITCHPTH
- removed SG1: F/QMBIII, buzzer:F/QMBIII
- removed U$1: ESP32_MINI_KIT, dedo:ESP32_MINI_KIT
- removed X1, X2, X3: 22-23-2021, con-molex:22-23-2021
- added CONECTOR1, JP2: (no value), pinhead:PINHD-1X2/90
- added LED1: (no value), led:LED5MM
- added PULSADOR: (no value), SparkFun-Retired:TAC_SWITCHPTH
- R1: device resistor:R-US_0207/7 -> resistor:R-US_0207/12
Connections:
- removed net N$17: X2-2.S
- removed net N$18: X2-1.S
- removed net N$19: X1-2.S
- removed net N$20: X1-1.S
- removed net N$21: SG1.-
- removed net N$22: LEFTQTR1A.2
- removed net N$23: RIGHTQTR1A.2
- removed net N$3: QTR8A.6
- removed net N$4: QTR8A.5
- removed net N$5: QTR8A.4
- removed net N$6: QTR8A.3
- removed net N$7: QTR8A.1
- removed net N$8: R1.2, S1.1, S1.2
- removed net VCC: X3-2.S
- net +5V: now also CONECTOR1.2, PULSADOR.1; no longer LEFTQTR1A.1, QTR8A.2, RIGHTQTR1A.1, S1.3, S1.4
- net GND: now also CONECTOR1.1, JP2.1, LED1.C; no longer LEFTQTR1A.3, R1.1, RIGHTQTR1A.3, SG1.+, X3-1.S
- net N$1: now also LED1.A, R1.2; no longer QTR8A.8
- net N$2: now also JP2.2, PULSADOR.3, R1.1; no longer QTR8A.7
Other:
- moved on the sheet: R1
