File: usainBotV2/usain_bot_chasis.brd (EAGLE design)
At the start: 100 x 80 mm, 10 parts, among them X1 22-23-2021, X2 22-23-2021, X3 22-23-2021

Commit message: carpetas ordenadas y limpias, proyectos de pcbs en este repo
Parts:
- removed U$1: ESP32_MINI_KIT, dedo:ESP32_MINI_KIT
- added ESP32: ESP32_MINI_KIT, dedo:ESP32_MINI_KIT
- moved LEFTQTR1A 82.9 mm to (-43.2, 66.0), turned to 90 degrees
- moved R1 75.8 mm to (-1.27, 17.8), turned to 90 degrees
- moved SG1 64.9 mm to (8.89, 17.8), turned to 90 degrees
- moved S1 56.0 mm to (-8.89, 16.5), turned to 270 degrees
- moved X1 39.2 mm to (-20.3, -10.2)
- moved X3 19.1 mm to (25.4, -10.2)
- moved RIGHTQTR1A 16.1 mm to (43.2, 66.0), turned to 90 degrees
- moved QTR8A 13.7 mm to (1.27, 44.5), turned to 180 degrees
Other:
- board size 100 x 80 mm -> 99 x 100.5 mm

Commit message: actualizado sensor cega y usain bot
Parts:
- removed X1, X2: 22-23-2021, con-molex:22-23-2021
- ESP32: device dedo:ESP32_MINI_KIT -> robot-hand:ESP32_MINI_KIT
Connections:
- net N$8 renamed BOTON
- removed net N$17: X2.2
- removed net N$18: X2.1
- removed net N$19: X1.2
- removed net N$20: X1.1
Changed lines of the file:
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@@
 <drawing>
 <settings>
-<setting alwaysvectorfont="no"/>
+<setting alwaysvectorfont="yes"/>
 <setting verticaltext="up"/>
 </settings>
@@
 <attribute name="VALUE" x="12.7" y="14.605" size="1.27" layer="27" ratio="10" rot="R90"/>
 </element>
-<element name="X1" library="con-molex" library_urn="urn:adsk.eagle:library:165" package="22-23-2021" package3d_urn="urn:adsk.eagle:package:8078633/1" value="22-23-2021" x="-20.32" y="-10.16" smashed="yes">
-<attribute name="MF" value="MOLEX" x="-20.32" y="-10.16" size="1.778" layer="27" display="off"/>
-<attribute name="MPN" value="22-23-2021" x="-20.32" y="-10.16" size="1.778" layer="27" display="off"/>
-<attribute name="NAME" x="-22.86" y="-6.35" size="1.016" layer="25" ratio="10"/>
-<attribute name="OC_FARNELL" value="1462926" x="-20.32" y="-10.16" size="1.778" layer="27" display="off"/>
-<attribute name="OC_NEWARK" value="25C3832" x="-20.32" y="-10.16" size="1.778" layer="27" display="off"/>
-<attribute name="VALUE" x="-22.86" y="-15.24" size="1.016" layer="27" ratio="10"/>
-</element>
-<element name="X2" library="con-molex" library_urn="urn:adsk.eagle:library:165" package="22-23-2021" package3d_urn="urn:adsk.eagle:package:8078633/1" value="22-23-2021" x="19.05" y="8.89" smashed="yes">
-<attribute name="MF" value="MOLEX" x="19.05" y="8.89" size="1.778" layer="27" display="off"/>
-<attribute name="MPN" value="22-23-2021" x="19.05" y="8.89" size="1.778" layer="27" display="off"/>
-<attribute name="NAME" x="16.51" y="12.7" size="1.016" layer="25" ratio="10"/>
-<attribute name="OC_FARNELL" value="1462926" x="19.05" y="8.89" size="1.778" layer="27" display="off"/>
-<attribute name="OC_NEWARK" value="25C3832" x="19.05" y="8.89" size="1.778" layer="27" display="off"/>
-<attribute name="VALUE" x="16.51" y="3.81" size="1.016" layer="27" ratio="10"/>
-</element>
 <element name="X3" library="con-molex" library_urn="urn:adsk.eagle:library:165" package="22-23-2021" package3d_urn="urn:adsk.eagle:package:8078633/1" value="22-23-2021" x="25.4" y="-10.16" smashed="yes">
 <attribute name="MF" value="MOLEX" x="25.4" y="-10.16" size="1.778" layer="27" display="off"/>
@@
 <attribute name="VALUE" x="22.86" y="-15.24" size="1.016" layer="27" ratio="10"/>
 </element>
-<element name="ESP32" library="dedo" package="ESP32_MINI_KIT" value="ESP32_MINI_KIT" x="0" y="-10.16" smashed="yes">
+<element name="ESP32" library="robot-hand" package="ESP32_MINI_KIT" value="ESP32_MINI_KIT" x="0" y="-10.16" smashed="yes">
 <attribute name="NAME" x="-15.078" y="2.589665625" size="1.27" layer="25"/>
 </element>
@@
 <signal name="N$6">
 <contactref element="QTR8A" pad="3"/>
-</signal>
-<signal name="N$17">
-<contactref element="X2" pad="2"/>
-</signal>
-<signal name="N$18">
-<contactref element="X2" pad="1"/>
-</signal>
-<signal name="N$19">
-<contactref element="X1" pad="2"/>
-</signal>
-<signal name="N$20">
-<contactref element="X1" pad="1"/>
 </signal>
 <signal name="GND">
@@
 <contactref element="X3" pad="1"/>
 <contactref element="R1" pad="1"/>
-<wire x1="-1.27" y1="13.97" x2="43.18" y2="68.58" width="0" layer="19" extent="1-1"/>
+<wire x1="8.89" y1="14.5288" x2="43.18" y2="68.58" width="0" layer="19" extent="1-1"/>
+<wire x1="-1.27" y1="13.97" x2="8.89" y2="14.5288" width="0" layer="19" extent="1-1"/>
+<wire x1="24.13" y1="-10.16" x2="8.89" y2="14.5288" width="0" layer="19" extent="1-1"/>
 <wire x1="-43.18" y1="68.58" x2="-1.27" y2="13.97" width="0" layer="19" extent="1-1"/>
-<wire x1="8.89" y1="14.5288" x2="-1.27" y2="13.97" width="0" layer="19" extent="1-1"/>
-<wire x1="24.13" y1="-10.16" x2="8.89" y2="14.5288" width="0" layer="19" extent="1-1"/>
 </signal>
 <signal name="+5V">
@@
 <contactref element="S1" pad="3"/>
 <contactref element="S1" pad="4"/>
-<wire x1="-43.18" y1="63.5" x2="43.18" y2="63.5" width="0" layer="19" extent="1-1"/>
-<wire x1="-11.1506" y1="19.7612" x2="-43.18" y2="63.5" width="0" layer="19" extent="1-1"/>
+<wire x1="7.62" y1="44.45" x2="43.18" y2="63.5" width="0" layer="19" extent="1-1"/>
+<wire x1="-11.1506" y1="19.7612" x2="7.62" y2="44.45" width="0" layer="19" extent="1-1"/>
 <wire x1="-11.1506" y1="13.2588" x2="-11.1506" y2="19.7612" width="0" layer="19" extent="1-1"/>
-<wire x1="7.62" y1="44.45" x2="-11.1506" y2="13.2588" width="0" layer="19" extent="1-1"/>
+<wire x1="-43.18" y1="63.5" x2="-11.1506" y2="19.7612" width="0" layer="19" extent="1-1"/>
 </signal>
 <signal name="VCC">
 <contactref element="X3" pad="2"/>
 </signal>
-<signal name="N$8">
+<signal name="BOTON">
 <contactref element="S1" pad="1"/>
 <contactref element="S1" pad="2"/>
@@
 <contactref element="QTR8A" pad="1"/>
 </signal>
+<signal name="N$9">
+</signal>
 </signals>
