File: Sensor CEGA/sensor.brd (EAGLE design)
At the start: 68.6 x 63.2 mm, 8 parts, among them J1 22-27-2021-02, J2 22-27-2031-03

Commit message: add libraries
Parts:
- renumbered J2 to TEMP_HUM, PARTICULAS to MP_SENSOR, U$1 to ARDUINO_PRO_MINI
Connections:
- net D10 renamed SD_CS
- net D11 renamed SD_SDO
- net D12 renamed SD_SDI
- net D13 renamed SD_SCK
Routing:
- net GND: track 129.8 -> 175.3 mm
- net +5V: track 193.2 -> 223.0 mm, vias 0 -> 1
- net D5: track 93.3 -> 99.1 mm
- net SD_SCK: track 46.9 -> 46.1 mm, vias 2 -> 1
